File: hardware/KiCAD_Template/standard.kicad_pcb (KiCad board)
At the start: 4 copper layers, 100 x 100 mm, 0 parts

Commit message: fix: kicad build automation output directory
Other:
- board text added: "0.2000 mm / 0.2000 mm"
- board text added: "0.3000 mm"
- board text added: "1.6000 mm"
- board text added: "100.0000 mm x 100.0000 mm"
- board text removed: "0.2 mm / 0.2 mm"
- board text removed: "0.3 mm"
- board text removed: "1.6 mm"
- board text removed: "100 mm x 100 mm"
